Commit message: test done

File: description/ros2_control.xacro (robot description, xacro)
@@ -1,27 +1,27 @@
 <?xml version="1.0"?>
 <robot xmlns:xacro="http://www.ros.org/wiki/xacro">
-    <ros2_control name = "Gazebo_System" type = "system">
+    <ros2_control name="GazeboSystem" type="system">
         <hardware>
-            <plugin>gazebo_ros2_control/Gazebo_System</plugin>
+            <plugin>gazebo_ros2_control/GazeboSystem</plugin>
         </hardware>
-        <joint name="left_wheel_joint" >
-            <command_interface name = "velocity">
-                <param name="min" value="-10"/>
-                <param name="max" value="10"/>
+        <joint name="left_wheel_joint">
+            <command_interface name="velocity">
+                <param name="min">-10</param>
+                <param name="max">10</param>
             </command_interface>
-            <state_interface name = "velocity"/>
-            <state_interface name = "position"/>
+            <state_interface name="position" />
+            <state_interface name="velocity" />
         </joint>
-        <joint name="right_wheel_joint" >
-            <command_interface name = "velocity">
-                <param name="min" value="-10"/>
-                <param name="max" value="10"/>
+        <joint name="right_wheel_joint">
+            <command_interface name="velocity">
+                <param name="min">-10</param>
+                <param name="max">10</param>
             </command_interface>
-            <state_interface name = "velocity"/>
-            <state_interface name = "position"/>
+            <state_interface name="velocity" />
+            <state_interface name="position" />
         </joint>
-    </ros2_control>
+``  </ros2_control>
     <gazebo>
-        <plugin filename = "libgazebo_ros2_control.so" name= "gazebo_ros2_control">
+        <plugin filename="libgazebo_ros2_control.so" name="gazebo_ros2_control">
             <parameters>$(find test_bot)/config/my_controller.yaml</parameters>
         </plugin>
